File: PCB_watch.kicad_sch (KiCad schematic)
At the start: 21 parts

Commit message: Rev0.0
Parts:
- removed C100, C? (x2): C, symbol Device:C
- removed J?: (no value), symbol Connector:AVR-UPDI-6
- removed NMOS_OPEN_DRAIN: MNMOS, symbol pspice:MNMOS
- removed R?, Rp: R, symbol Device:R
- removed SW100: (no value), symbol Switch:SW_Push
- removed U?: PT7C4563BQ1WEX, symbol PCB_watch_symbol_lib:PT7C4563BQ1WEX
- removed U?: 5V_to_3V3_DCDC_Converter, symbol PCB_watch_symbol_lib:5V_to_3V3_DCDC_Converter
- removed U?: XDBCZLNDMD-0.032768, symbol PCB_watch_symbol_lib:XDBCZLNDMD-0.032768
- added BT101, BT102: (no value), 9V_battery_coin:S8211-46R, symbol Device:Battery_Cell
- added BT201: CR2302, 9V_battery_coin:S8211-46R, symbol Device:Battery_Cell
- added C201, C301, C302: (no value), symbol Device:C
- added C202: (no value), Capacitor_SMD:C_0805_2012Metric_Pad1.18x1.45mm_HandSolder, symbol Device:C
- added C203: 10uF, Capacitor_SMD:C_0805_2012Metric_Pad1.18x1.45mm_HandSolder, symbol Device:C
- added CRYS101, CRYS201: CRYSTAL 32.768KHZ HC-49U, symbol PCB_watch_symbol_lib:CRYSTAL 32.768KHZ HC-49U
- added RTC101: DS1307+, Package_DIP:DIP-8_W7.62mm, symbol Timer_RTC:DS1307+
- added Rp_i2c_202: 2K, Resistor_SMD:R_0805_2012Metric_Pad1.20x1.40mm_HandSolder, symbol Device:R
- added SW101: (no value), symbol Switch:SW_SPDT
- C101, C102: value C -> (none)
- CONN101: renamed from J?; value (none) -> Conn_01x04_Male
- FB101: renamed from FB100; value (none) -> Ferrite Bead
- ISP101: renamed from J?; value (none) -> AVR-ISP-6
- uC101: renamed from U?; value (none) -> ATmega88-20A; footprint (none) -> Package_QFP:TQFP-32_7x7mm_P0.8mm
- gave numbers to parts that had none: 1
- renumbered D100 to D101, F100 to F101, Rp to Rp_i2c_201
Connections:
- net uC VCC is gone; now on net VCC: FB101.2, uC101.18 (AVCC), uC101.4 (VCC), uC101.6 (VCC)
- net GND: now also BT101.2 (-), BT201.2 (-), C201.2, C202.2, C203.2, C301.2, C302.2, RTC101.4 (GND), SW101.1 (A)
- net LCD_SCL: now also uC101.28 (PC5), RTC101.6 (SCL), Rp_i2c_202.2
- net LCD_SDA: now also Rp_i2c_201.2, uC101.27 (PC4), RTC101.5 (SDA)
- net VCC: now also C201.1, C202.1, C203.1, RTC101.8 (VCC), Rp_i2c_202.1
- net X1: now also CRYS101.1 (X1), RTC101.1 (X1)
- net X2: now also CRYS101.2 (X2), RTC101.2 (X2)
- net at FB101.1: now also C101.1, F101.2; no longer D101.1 (K)
- net at D101.2 (A): now also SW101.3 (C); no longer F101.2
- net MISO: now reaches ISP101.1 (MISO)
- net MISO: now also uC101.16 (PB4)
- net SCK: now reaches ISP101.3 (SCK)
- net SCK: now also uC101.17 (PB5)
- net MOSI: now reaches ISP101.4 (MOSI)
- net MOSI: now also uC101.15 (PB3)
- net ~{RST}: now reaches ISP101.5 (~{RST})
- net ~{RST}: now also uC101.29 (~{RESET}/PC6)
- net XTAL1: now reaches uC101.7 (XTAL1/PB6)
- net XTAL1: now also C301.1, CRYS201.1 (X1)
- net XTAL2: now reaches uC101.8 (XTAL2/PB7)
- net XTAL2: now also C302.1, CRYS201.2 (X2)
- net 5V: no longer names the net of F101.1
- net 5V: now also D101.1 (K)
- new net: BT201.1 (+), RTC101.3 (VBAT)
- new net: BT102.1 (+), SW101.2 (B)
- new net: BT101.1 (+), BT102.2 (-)
- no-connect marks 1 -> 18
Other:
- note added: "ISP Connector"
- note added: "Microcontroller"
- note added: "PB: SPI"
- note added: "PC: I2C"
- note added: "PD: USART"
- note added: "Real Time Clock, and Crystal Oscillator"
- note added: "Voltage Supply Filtering, and Resistor Drop"
- note removed: "External Connector"
- company: (none) -> Rajnesh Joshi
- title: (none) -> PCB Watch [Draft]
- moved on the sheet: CONN101, D101, F101, FB101, ISP101, LCD101, Rp_i2c_201, uC101
